File: LIU.kicad_pcb (KiCad board)
At the start: 2 copper layers, 100 x 100 mm, 116 parts, among them J1 Audio Input, J2 Audio Input, J3 UHF out, J4 UHF in, J5 12 Volts Input, J6 VHF in, J7 VHF out, J8 Audio Out, J9 Audio Out, Q1 2N7002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

Commit message: Further layout work
Parts:
- C15, C16, C17, C18, C7: moved to B.Cu
- moved J6 136.2 mm to (82.7, 93.8)
- moved J7 127.8 mm to (82.7, 104.8)
- moved C15 91.7 mm to (121.6, 129.8), turned to 270 degrees
- moved C11 90.0 mm to (133.8, 82.7), turned to 90 degrees
- moved R1 87.3 mm to (122.5, 67.2)
- moved C16 85.6 mm to (121.6, 135.2), turned to 270 degrees
- moved C2 84.4 mm to (120.3, 76.3)
- moved C6 83.2 mm to (122.5, 108.5)
- moved C7 78.6 mm to (114.0, 120.9), turned to 270 degrees
- moved C14 71.5 mm to (132.3, 102.0)
- moved C13 67.2 mm to (132.5, 107.2)
- moved R7 65.5 mm to (129.1, 76.8)
- moved R13 60.2 mm to (133.0, 97.2)
- moved C18 57.4 mm to (121.6, 119.7), turned to 270 degrees
- moved C8 52.3 mm to (100.1, 98.1)
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
Commit message: All components on the board
Parts:
- C13, C14, C6, C8, C9: moved to B.Cu
- J1, J2: value Audio Input -> Audio In
- J8, J9: value Audio Out -> Audio Output
- moved R9 108.3 mm to (141.6, 67.3), turned to 90 degrees
- moved C9 97.7 mm to (115.6, 143.2), turned to 180 degrees
- moved C22 92.1 mm to (148.5, 65.2), turned to 270 degrees
- moved C3 83.3 mm to (111.5, 125.3), turned to 270 degrees
- moved D2 83.2 mm to (136.1, 53.9), turned to 180 degrees
- moved C21 82.6 mm to (132.3, 126.2), turned to 90 degrees
- moved J4 76.7 mm to (139.2, 60.8), turned to 180 degrees
- moved Q2 68.8 mm to (135.9, 67.2), turned to 90 degrees
- moved J7 66.9 mm to (133.0, 60.8), turned to 180 degrees
- moved C23 66.8 mm to (138.0, 80.2), turned to 90 degrees
- moved R2 66.5 mm to (111.9, 115.2), turned to 90 degrees
- moved D1 66.4 mm to (112.8, 53.9)
- moved C24 65.2 mm to (138.0, 123.1), turned to 270 degrees
- moved R12 60.8 mm to (129.8, 132.1), turned to 180 degrees
- moved R18 59.7 mm to (129.7, 67.7), turned to 270 degrees
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Connections:
- D1 pad 1: Net-(D1-Pad1) -> GND
- D1 pad 2: +5v -> Net-(D1-Pad2)
- D2 pad 1: Net-(D2-Pad1) -> GND
- D2 pad 2: +5v -> Net-(D2-Pad2)
- J1 pad 1: Net-(J1-Pad1) -> GND
- J1 pad 2: GND -> Net-(J1-Pad2)
- J2 pad 1: Net-(J2-Pad1) -> GND
- J2 pad 2: GND -> Net-(J2-Pad2)
- J3 pad 1: Net-(J3-Pad1) -> GND
- J3 pad 2: GND -> Net-(J3-Pad2)
- J4 pad 1: Net-(J4-Pad1) -> GND
- J4 pad 2: GND -> Net-(J4-Pad2)
- J6 pad 1: Net-(J3-Pad1) -> GND
- J6 pad 2: GND -> Net-(J3-Pad2)
- J7 pad 1: Net-(J4-Pad1) -> GND
- J7 pad 2: GND -> Net-(J4-Pad2)
- JP1 pad 2: Net-(J1-Pad1) -> Net-(J1-Pad2)
- JP2 pad 2: Net-(J2-Pad1) -> Net-(J2-Pad2)
- Q1 pad 1: Net-(J4-Pad1) -> Net-(J4-Pad2)
- Q1 pad 3: Net-(Q1-Pad3) -> Net-(D1-Pad2)
- Q2 pad 1: Net-(J3-Pad1) -> Net-(J3-Pad2)
- Q2 pad 3: Net-(Q2-Pad3) -> Net-(D2-Pad2)
- R10 pad 2: Net-(J4-Pad1) -> Net-(J4-Pad2)
- R15 pad 1: Net-(D1-Pad1) -> Net-(D1-Pad2)
- R15 pad 2: Net-(Q1-Pad3) -> +5v
- R17 pad 1: Net-(R17-Pad1) -> Net-(C26-Pad2)
- R17 pad 2: Net-(C26-Pad2) -> Net-(R17-Pad2)
- R18 pad 1: Net-(D2-Pad1) -> Net-(D2-Pad2)
- R18 pad 2: Net-(Q2-Pad3) -> +5v
- R9 pad 2: Net-(J3-Pad1) -> Net-(J3-Pad2)
- RV4 pad 2: Net-(R17-Pad1) -> Net-(R17-Pad2)

Commit message: Further PCB layout
Parts:
- moved R10 34.1 mm to (141.5, 67.6)
- moved D1 23.2 mm to (135.9, 53.9), turned to 180 degrees
- moved D2 23.0 mm to (113.2, 53.9)
- moved Q1 22.7 mm to (135.9, 67.1)
- moved Q2 22.7 mm to (113.2, 67.2)
- moved R18 22.3 mm to (107.5, 67.5)
- moved R9 22.0 mm to (119.7, 67.5)
- moved R15 10.1 mm to (129.8, 67.6)
Routing:
- net +5v: track 3.14 -> 69.9 mm
- net GND: track 924.1 -> 982.0 mm
- net Net-(J3-Pad2): track 0.00 -> 29.4 mm
- net Net-(J4-Pad2): track 0.00 -> 29.1 mm
- net Net-(D1-Pad2): track 0.00 -> 23.7 mm
- net Net-(D2-Pad2): track 0.00 -> 23.5 mm

Commit message: Project completed
Parts:
- moved R5 4.81 mm to (175.4, 68.9), turned to 270 degrees
- turned R17 to 0 degrees
Routing:
- net GND: track 982.0 -> 1132.9 mm, vias 0 -> 40
- net +5v: track 69.9 -> 157.0 mm
- net Net-(C25-Pad1): track 55.1 -> 88.0 mm, vias 0 -> 2
- net Net-(JP1-Pad1): track 0.00 -> 30.5 mm, vias 0 -> 1
- net Net-(JP1-Pad3): track 0.00 -> 26.5 mm
- net Net-(JP2-Pad3): track 0.00 -> 26.2 mm, vias 0 -> 2
- net Net-(C21-Pad2): track 0.00 -> 18.3 mm
- net Net-(J2-Pad2): track 0.00 -> 18.0 mm
- net Net-(C12-Pad1): track 0.00 -> 16.0 mm
- net Net-(J1-Pad2): track 0.00 -> 15.7 mm
- net Net-(C11-Pad1): track 0.00 -> 15.3 mm
- net Net-(JP3-Pad2): track 0.00 -> 14.2 mm
- net Net-(R17-Pad1): track 13.0 -> 0.00 mm
- net Net-(JP4-Pad2): track 0.00 -> 12.4 mm
- net Net-(R17-Pad2): track 0.00 -> 11.0 mm
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